File: pcb/M5StackSideBB.sch (KiCad schematic (older format))
At the start: 4 parts, among them J1 Conn_01x14, J2 Conn_01x14, J3 Conn_02x15_Odd_Even, J4 Conn_02x15_Odd_Even

Commit message: Change footprint for top pad without THT holes
Parts:
- J3: footprint footprints:PinHeader_2x15_P2.54mm_Vertical_SMD_for_M5Stack_top_only_round_pads -> footprints:PinHeader_2x15_P2.54mm_SMD_pads_only
Changed lines of the file:
@@
 F 0 "J3" H 8150 3917 50  0000 C CNN
 F 1 "Conn_02x15_Odd_Even" H 8150 3826 50  0000 C CNN
-F 2 "footprints:PinHeader_2x15_P2.54mm_Vertical_SMD_for_M5Stack_top_only_round_pads" H 8100 3000 50  0001 C CNN
+F 2 "footprints:PinHeader_2x15_P2.54mm_SMD_pads_only" H 8100 3000 50  0001 C CNN
 F 3 "~" H 8100 3000 50  0001 C CNN
 	1    8100 3000

Commit message: Apply smaller pads for top and bottom
Parts:
- J4: footprint footprints:PinSocket_2x15_P2.54mm_Vertical_SMD_for_M5Stack_bottom -> footprints:PinSocket_2x15_P2.54mm_Vertical_SMD_just_for_M5Stack_bottom
Changed lines of the file:
@@
 F 0 "J4" H 8150 6017 50  0000 C CNN
 F 1 "Conn_02x15_Odd_Even" H 8150 5926 50  0000 C CNN
-F 2 "footprints:PinSocket_2x15_P2.54mm_Vertical_SMD_for_M5Stack_bottom" H 8100 5100 50  0001 C CNN
+F 2 "footprints:PinSocket_2x15_P2.54mm_Vertical_SMD_just_for_M5Stack_bottom" H 8100 5100 50  0001 C CNN
 F 3 "~" H 8100 5100 50  0001 C CNN
 	1    8100 5100

Commit message: Add bottom pads for spacer PCB
Parts:
- J3: footprint footprints:PinHeader_2x15_P2.54mm_SMD_pads_only -> footprints:PinHeader_2x15_P2.54mm_M5Stack_SpacerPCB_pads
Changed lines of the file:
@@
 F 0 "J3" H 8150 3917 50  0000 C CNN
 F 1 "Conn_02x15_Odd_Even" H 8150 3826 50  0000 C CNN
-F 2 "footprints:PinHeader_2x15_P2.54mm_SMD_pads_only" H 8100 3000 50  0001 C CNN
+F 2 "footprints:PinHeader_2x15_P2.54mm_M5Stack_SpacerPCB_pads" H 8100 3000 50  0001 C CNN
 F 3 "~" H 8100 3000 50  0001 C CNN
 	1    8100 3000
