File: spacer_pcb/spacer_pcb.sch (KiCad schematic (older format))
At the start: 3 parts, among them J1 Conn_01x15, J2 Conn_02x15_Odd_Even, J3 Conn_01x15

Commit message: Assign new footprint for spacer
Parts:
- J2: footprint Connector_PinHeader_2.54mm:PinHeader_2x15_P2.54mm_Vertical_SMD -> footprints:PinHeader_2x15_P2.54mm_Vertical_SMD_for_M5Stack
Changed lines of the file:
@@
 F 0 "J2" H 6450 4517 50  0000 C CNN
 F 1 "Conn_02x15_Odd_Even" H 6450 4426 50  0000 C CNN
-F 2 "Connector_PinHeader_2.54mm:PinHeader_2x15_P2.54mm_Vertical_SMD" H 6400 3600 50  0001 C CNN
+F 2 "footprints:PinHeader_2x15_P2.54mm_Vertical_SMD_for_M5Stack" H 6400 3600 50  0001 C CNN
 F 3 "~" H 6400 3600 50  0001 C CNN
 	1    6400 3600

Commit message: Add bottom pads for spacer PCB
Parts:
- removed J1, J3: Conn_01x15, Connector_PinHeader_2.54mm:PinHeader_1x15_P2.54mm_Vertical, symbol Connector_Generic:Conn_01x15
- J2: footprint footprints:PinHeader_2x15_P2.54mm_Vertical_SMD_for_M5Stack -> footprints:PinHeader_2x15_P2.54mm_M5Stack_SpacerPCB
Connections:
- no-connect marks 0 -> 30
Changed lines of the file:
@@
 F 0 "J2" H 6450 4517 50  0000 C CNN
 F 1 "Conn_02x15_Odd_Even" H 6450 4426 50  0000 C CNN
-F 2 "footprints:PinHeader_2x15_P2.54mm_Vertical_SMD_for_M5Stack" H 6400 3600 50  0001 C CNN
+F 2 "footprints:PinHeader_2x15_P2.54mm_M5Stack_SpacerPCB" H 6400 3600 50  0001 C CNN
 F 3 "~" H 6400 3600 50  0001 C CNN
 	1    6400 3600
 	1    0    0    -1
 $EndComp
-$Comp
-L Connector_Generic:Conn_01x15 J3
-U 1 1 5B3F1ECC
-P 6900 3600
-F 0 "J3" H 6850 4550 50  0000 L CNN
-F 1 "Conn_01x15" H 6700 4450 50  0000 L CNN
-F 2 "Connector_PinHeader_2.54mm:PinHeader_1x15_P2.54mm_Vertical" H 6900 3600 50  0001 C CNN
-F 3 "~" H 6900 3600 50  0001 C CNN
-	1    6900 3600
-	1    0    0    -1
-$EndComp
-$Comp
-L Connector_Generic:Conn_01x15 J1
-U 1 1 5B3F1F26
-P 6000 3600
-F 0 "J1" H 5920 4517 50  0000 C CNN
-F 1 "Conn_01x15" H 5920 4426 50  0000 C CNN
-F 2 "Connector_PinHeader_2.54mm:PinHeader_1x15_P2.54mm_Vertical" H 6000 3600 50  0001 C CNN
-F 3 "~" H 6000 3600 50  0001 C CNN
-	1    6000 3600
-	-1   0    0    -1
-$EndComp
+NoConn ~ 6200 2900
+NoConn ~ 6200 3000
+NoConn ~ 6200 3100
+NoConn ~ 6200 3200
+NoConn ~ 6200 3300
+NoConn ~ 6200 3400
+NoConn ~ 6200 3500
+NoConn ~ 6200 3600
+NoConn ~ 6200 3700
+NoConn ~ 6200 3800
+NoConn ~ 6200 3900
+NoConn ~ 6200 4000
+NoConn ~ 6200 4100
+NoConn ~ 6200 4200
+NoConn ~ 6200 4300
+NoConn ~ 6700 4300
+NoConn ~ 6700 4200
+NoConn ~ 6700 4100
+NoConn ~ 6700 4000
+NoConn ~ 6700 3900
+NoConn ~ 6700 3800
+NoConn ~ 6700 3700
+NoConn ~ 6700 3600
+NoConn ~ 6700 3500
+NoConn ~ 6700 3400
+NoConn ~ 6700 3300
+NoConn ~ 6700 3200
+NoConn ~ 6700 3100
+NoConn ~ 6700 3000
+NoConn ~ 6700 2900
 $EndSCHEMATC
